File: Lab Supply.kicad_pcb (KiCad board)
At the start: 2 copper layers, 198.1 x 116.8 mm, 73 parts, among them M1 Fan_4pin, Q1 TIP121, Q2 2N3904, Q3 TIP121, Q5 2N3904, SW1 ENABLE, U1 LM324, U2 LM7812_TO220, U3 MCP4922, U4 LM7805_TO220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

Commit message: Added README
Parts:
- added ?: MountingHole_3.2mm_M3, MountingHole:MountingHole_3.2mm_M3, F.Cu at (177.8, 39.5)
- added C14: 100n, Capacitor_THT:C_Rect_L10.0mm_W2.5mm_P7.50mm_MKS4, F.Cu at (93.0, 114.0)
- added C17: 10u, Capacitor_THT:CP_Radial_D8.0mm_P3.50mm, F.Cu at (94.3, 124.5)
- added C18: 100n, Capacitor_THT:C_Rect_L10.0mm_W2.5mm_P7.50mm_MKS4, F.Cu at (128.2, 110.1)
- added LCD: Display, Connector_PinHeader_2.54mm:PinHeader_1x04_P2.54mm_Vertical, F.Cu at (126.5, 145.8)
- added R26: 47k, Resistor_THT:R_Axial_DIN0204_L3.6mm_D1.6mm_P7.62mm_Horizontal, F.Cu at (109.2, 98.7)
- added REF**: MountingHole_3.2mm_M3, MountingHole:MountingHole_3.2mm_M3, F.Cu at (177.8, 148.5)
- added REF**: MountingHole_3.2mm_M3, MountingHole:MountingHole_3.2mm_M3, F.Cu at (51.1, 39.5)
- added REF**: MountingHole_3.2mm_M3, MountingHole:MountingHole_3.2mm_M3, F.Cu at (51.1, 148.5)
- CURRENT: renamed from H1; footprint Arduino:5 Pin Header -> Connector_PinHeader_2.54mm:PinHeader_1x05_P2.54mm_Vertical
- R4: value 68k -> 47k
- RV5: value 200k -> 20k
- VOLTAGE: renamed from H2; footprint Arduino:5 Pole Header -> Connector_PinHeader_2.54mm:PinHeader_1x05_P2.54mm_Vertical
- moved R4 295.9 mm to (132.1, 61.0)
- moved Q1 293.0 mm to (154.8, 39.0), turned to 0 degrees
- moved R11 290.4 mm to (113.5, 60.7), turned to -90 degrees
- moved V+ 275.9 mm to (174.8, 76.6)
- moved V- 274.5 mm to (174.6, 109.6)
- moved SW1 269.0 mm to (136.8, 44.7), turned to 0 degrees
- moved U3 266.1 mm to (92.2, 86.1)
- moved R7 265.9 mm to (166.9, 88.4), turned to -90 degrees
- moved C1 258.9 mm to (158.9, 90.6), turned to -90 degrees
- moved VOLTAGE 256.1 mm to (135.0, 112.0)
- moved U6 254.9 mm to (118.4, 91.2)
- moved C9 254.5 mm to (92.5, 107.7)
- moved U7 253.0 mm to (114.3, 124.5)
- moved CURRENT 252.9 mm to (134.4, 132.1)
- moved R20 248.0 mm to (103.9, 91.1), turned to -90 degrees
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- renumbered CONN3 to AC1, CONN4 to AC2, CONN1 to V+, CONN2 to V-
Connections:
- Q1 pad 1: +28V -> Net-(D11-A)
- Q1 pad 2: Net-(D11-A) -> +28V
- Q3 pad 1: +36V -> Net-(D9-K)
- Q3 pad 2: Net-(D9-K) -> +36V
- SW1 pad 1: Net-(D11-K) -> Net-(SW1-A)
- U1 pad 12: V_VSET -> Net-(SW1-A)
- U3 pad 3: unconnected-(U3-~{CS}-Pad3) -> Net-(U3-~{CS})
- U7 pad 21: unconnected-(U7-SDA-Pad21) -> Net-(H3-SDA)
- U7 pad 22: unconnected-(U7-SCL-Pad22) -> Net-(H3-SCL)
- U7 pad 29: unconnected-(U7-D13-Pad29) -> Net-(U3-~{CS})
- U7 pad 31: unconnected-(U7-GND-Pad31) -> GND
Routing:
- net +5V: track 0.00 -> 255.9 mm, vias 0 -> 2
- net +28V: track 0.00 -> 219.1 mm, vias 0 -> 1
- net +36V: track 0.00 -> 172.6 mm
- net Net-(U3-SCK): track 0.00 -> 153.1 mm, vias 0 -> 3
- net ISENSE: track 0.00 -> 151.1 mm
- net V+: track 0.00 -> 124.7 mm, vias 0 -> 2
- net Net-(U6-DOUT): track 0.00 -> 92.2 mm, vias 0 -> 1
- net Net-(D12-A): track 0.00 -> 90.1 mm, vias 0 -> 2
- net Net-(D11-A): track 0.00 -> 89.4 mm, vias 0 -> 2
- net Net-(SW1-A): track 0.00 -> 79.1 mm
- net Net-(U3-SDI): track 0.00 -> 73.8 mm, vias 0 -> 2
- net V_ISET: track 0.00 -> 68.8 mm, vias 0 -> 2
- net Net-(R14-Pad2): track 0.00 -> 63.8 mm, vias 0 -> 2
- net Net-(U3-~{CS}): track 0.00 -> 59.9 mm, vias 0 -> 2
- net Net-(D9-K): track 0.00 -> 54.3 mm, vias 0 -> 3
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- added copper zone on B.Cu, net GND
Other:
- board size 198.1 x 116.8 mm -> 134.9 x 116.8 mm
- board text added: "https://github.com/prydin/lab-supply V1.0 Nov 2023"

Commit message: Corrected reversed display header
Parts:
- SHUTDOWN: renamed from SW1; footprint Arduino:2 Pin Header -> Connector_PinHeader_2.54mm:PinHeader_1x02_P2.54mm_Vertical
- moved H3 10.2 mm to (126.5, 135.6), turned to 0 degrees
- moved R13 5.18 mm to (78.2, 100.6)
- moved SHUTDOWN 5.14 mm to (137.4, 49.8)
- moved U2 3.86 mm to (76.5, 117.3)
- moved C4 3.30 mm to (55.2, 63.8)
- moved C5 3.30 mm to (55.2, 83.8)
- moved C6 3.30 mm to (55.2, 104.1)
- renumbered CURRENT to H1, VOLTAGE to H2, LCD to H3
Routing:
- net Net-(H3-SDA): track 4.99 -> 12.4 mm
- net +36V: track 172.6 -> 178.9 mm
- net Net-(H3-SCL): track 4.99 -> 7.99 mm
- net Net-(M1-+): track 28.0 -> 25.3 mm
- net +28V: track 219.1 -> 221.8 mm
- net +5V: track 255.9 -> 254.1 mm
- net Net-(H1-CLK): track 15.6 -> 17.0 mm
Other:
- board text added: "+5V"
- board text added: "CLK"
- board text added: "DT"
- board text added: "GND"
- board text added: "SCL"
- board text added: "SDA"
- board text added: "SW"
- board text added: "https://github.com/prydin/lab-supply V1.1 Nov 2023"
- board text removed: "https://github.com/prydin/lab-supply V1.0 Nov 2023"

Commit message: WIP
Parts:
- removed R13: 100, Resistor_THT:R_Axial_DIN0204_L3.6mm_D1.6mm_P7.62mm_Horizontal
- added AC1: AC1, Connector_Wire:SolderWire-1.5sqmm_1x01_D1.7mm_OD3.9mm, F.Cu at (57.0, 120.0)
- added C19: 10u, Capacitor_THT:CP_Radial_D8.0mm_P3.50mm, F.Cu at (83.5, 104.0)
- added C7: 100n, Capacitor_THT:C_Rect_L10.0mm_W2.5mm_P7.50mm_MKS4, F.Cu at (54.2, 105.0)
- added D1: POWER, Connector_PinHeader_2.54mm:PinHeader_1x02_P2.54mm_Vertical, F.Cu at (147.1, 51.6)
- added R27: 10k, Resistor_THT:R_Axial_DIN0204_L3.6mm_D1.6mm_P7.62mm_Horizontal, F.Cu at (117.1, 131.1)
- added R28: 1.5k, Resistor_THT:R_Axial_DIN0204_L3.6mm_D1.6mm_P7.62mm_Horizontal, F.Cu at (142.0, 46.7)
- added TH1: 10k NTC, Connector_PinHeader_2.54mm:PinHeader_1x02_P2.54mm_Vertical, F.Cu at (128.3, 124.2)
- C6: value 4700u -> 100n; footprint Capacitor_THT:CP_Radial_D18.0mm_P7.50mm -> Capacitor_THT:C_Rect_L10.0mm_W2.5mm_P7.50mm_MKS4
- moved C6 6.22 mm to (54.2, 98.0)
- moved C3 4.57 mm to (92.3, 38.7)
- moved U4 4.07 mm to (79.2, 39.1)
- moved M1 2.30 mm to (89.5, 136.0)
- renumbered SHUTDOWN to SW1
Connections:
- C4 pad 2: GND -> CENTER
- C5 pad 1: +36V -> CENTER
- C6 pad 2: GND -> CENTER
- M1 pad 3: unconnected-(M1-Tacho-Pad3) -> Net-(M1-Tacho)
- U2 pad 1: +28V -> CENTER
- U4 pad 1: +28V -> CENTER
- U7 pad 17: unconnected-(U7-D6-Pad17) -> Net-(M1-PWM)
- U7 pad 18: unconnected-(U7-D4-Pad18) -> Net-(M1-Tacho)
- U7 pad 21: Net-(H3-SDA) -> unconnected-(U7-D1-Pad21)
- U7 pad 22: Net-(H3-SCL) -> Net-(H3-SDA)
- U7 pad 23: Net-(H1-CLK) -> Net-(H3-SCL)
- U7 pad 24: Net-(H1-DT) -> Net-(H1-CLK)
- U7 pad 25: Net-(H1-SW) -> Net-(H1-DT)
- U7 pad 26: Net-(H2-CLK) -> Net-(H1-SW)
- U7 pad 27: Net-(H2-DT) -> Net-(H2-CLK)
- U7 pad 28: Net-(H2-SW) -> Net-(H2-DT)
- U7 pad 29: Net-(U3-~{CS}) -> Net-(H2-SW)
- U7 pad 30: unconnected-(U7-VBUS-Pad30) -> Net-(U3-~{CS})
- U7 pad 31: GND -> unconnected-(U7-VBUS-Pad31)
- U7 pad 32: (no net) -> GND
- U7 pad 5: unconnected-(U7-A0-Pad5) -> Net-(U7-A0)
Routing:
- net CENTER: track 0.00 -> 153.9 mm
- net +28V: track 221.8 -> 143.3 mm
- net Net-(U7-A0): track 0.00 -> 32.6 mm, vias 0 -> 2
- net Net-(M1-Tacho): track 0.00 -> 31.5 mm, vias 0 -> 1
- net Net-(M1-PWM): track 0.00 -> 19.7 mm
- net +36V: track 178.9 -> 196.0 mm
- net +5V: track 254.1 -> 267.1 mm
- net Net-(M1-+): track 25.3 -> 37.2 mm
- net Net-(D1-A): track 0.00 -> 7.44 mm
- net Net-(H3-SCL): track 7.99 -> 14.9 mm
- net Net-(H3-SDA): track 12.4 -> 6.04 mm
- net Net-(U3-~{CS}): track 59.9 -> 55.0 mm
- net Net-(H2-SW): track 15.2 -> 13.6 mm
- net Net-(H2-CLK): track 15.2 -> 14.0 mm
- net Net-(H2-DT): track 15.2 -> 14.0 mm
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Other:
- board text added: "R"
- board text added: "https://github.com/prydin/lab-supply V1.2 Nov 2023"
- board text removed: "https://github.com/prydin/lab-supply V1.1 Nov 2023"

Commit message: WIP
Parts:
- Q2, Q5: footprint Package_TO_SOT_THT:TO-92_HandSolder -> Package_TO_SOT_THT:TO-92_Inline
- R7: value 3.9k -> 8.2k
Connections:
- C15 pad 1: Net-(U5-A) -> VREF
- C16 pad 1: GND -> VREF
- C16 pad 2: Net-(U5-A) -> GND
- Q2 pad 1: Net-(D11-K) -> GND
- Q2 pad 3: GND -> Net-(D11-K)
- Q5 pad 1: +28V -> Net-(Q5-E)
- Q5 pad 3: Net-(Q5-E) -> +28V
- R1 pad 2: Net-(U5-A) -> VREF
- U5 pad 1: GND -> VREF
- U5 pad 2: Net-(U5-A) -> GND
- U6 pad 8: Net-(U5-A) -> VREF
- U7 pad 1: GND -> unconnected-(U7-RST-Pad1)
Routing:
- net VREF: track 39.8 -> 109.0 mm
- net Net-(U5-A): track 51.7 -> 0.00 mm, vias 1 -> 0
- net Net-(Q5-B): track 24.1 -> 30.5 mm, vias 2 -> 0
- net Net-(Q5-E): track 13.6 -> 16.6 mm, vias 2 -> 0
- net +28V: track 143.3 -> 144.6 mm, vias 1 -> 0
- net Net-(Q2-B): track 17.4 -> 16.8 mm
- net Net-(D11-K): track 41.6 -> 42.1 mm
