File: Lab Supply.kicad_sch (KiCad schematic)
At the start: 80 parts, among them J1 V+, J2 V-, M1 Fan_4pin, Q1 TIP121, Q2 2N3904, Q3 TIP121, Q5 2N3904, SW1 ENABLE, T1 115V to 24V, U1 LM324, U2 LM7812_TO220, U3 MCP4922, U4 LM7805_TO220, U5 LM4040DBZ-2.0, U6 MCP3202

Commit message: Added README
Parts:
- removed Q1, Q3: TIP121, Package_TO_SOT_THT:TO-220-3_Vertical, symbol Simulation_SPICE:NPN
- added C14, C18: 100n, Capacitor_THT:C_Rect_L10.0mm_W2.5mm_P7.50mm_MKS4, symbol Device:C
- added C17: 10u, Capacitor_THT:CP_Radial_D8.0mm_P3.50mm, symbol Device:C_Polarized
- added H3: Display, Connector_PinHeader_1.00mm:PinHeader_1x04_P1.00mm_Vertical, symbol Headers:I2C Header
- added Q1, Q3: TIP121, Package_TO_SOT_THT:TO-220-3_Vertical, symbol Transistor_BJT:TIP121
- added R26: 47k, Resistor_THT:R_Axial_DIN0204_L3.6mm_D1.6mm_P7.62mm_Horizontal, symbol Device:R
- R4: value 68k -> 47k
- RV5: value 200k -> 20k
Connections:
- net +28V: now also Q1.2 (C), Q3.3 (E)
- net +36V: now also Q3.2 (C)
- net +5V: now also C14.1, C17.1, C18.1, H3.2 (+5V)
- net GND: now also C14.2, C17.2, C18.2, H3.1 (GND)
- net V+: now also Q1.3 (E)
- net V_VSET: now also R26.1; no longer U1.12 (+)
- net at D11.2 (A), D2.2 (A), R10.2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: now also Q1.1 (B)
- net at D11.1 (K), Q2.1 (C): no longer SW1.1 (A)
- net at C11.1, D9.1 (K), R12.2: now also Q3.1 (B)
- net at U7.21 (SDA): now also H3.3 (SDA)
- net at U7.22 (SCL): now also H3.4 (SCL)
- new net: R26.2, SW1.1 (A), U1.12 (+)
Other:
- moved on the sheet: R12

Commit message: WIP
Parts:
- added C19: 10u, Capacitor_THT:CP_Radial_D8.0mm_P3.50mm, symbol Device:C_Polarized
- added D1: POWER, Connector_PinHeader_2.54mm:PinHeader_1x02_P2.54mm_Vertical, symbol Device:LED
- added R27: 10k, Resistor_THT:R_Axial_DIN0204_L3.6mm_D1.6mm_P7.62mm_Horizontal, symbol Device:R
- added R28: 1.5k, Resistor_THT:R_Axial_DIN0204_L3.6mm_D1.6mm_P7.62mm_Horizontal, symbol Device:R
- added R29: 10, symbol Device:R
- added TH1: 10k NTC, Connector_PinHeader_2.54mm:PinHeader_1x02_P2.54mm_Vertical, symbol Device:Thermistor
- added V4: VSIN, symbol Simulation_SPICE:VSIN
- H1: footprint Arduino:5 Pin Header -> Connector_PinHeader_2.54mm:PinHeader_1x05_P2.54mm_Vertical
- H2: footprint Arduino:5 Pole Header -> Connector_PinHeader_2.54mm:PinHeader_1x05_P2.54mm_Vertical
- H3: footprint Connector_PinHeader_1.00mm:PinHeader_1x04_P1.00mm_Vertical -> Connector_PinHeader_2.54mm:PinHeader_1x04_P2.54mm_Vertical
- RLOAD1: value 100k -> 10k
- SW1: footprint Arduino:2 Pin Header -> Connector_PinHeader_2.54mm:PinHeader_1x02_P2.54mm_Vertical
Connections:
- net +28V: now also R28.1
- net +5V: now also TH1.1
- net GND: now also U7.32 (GND), C19.2, D1.1 (K), R27.2
- net ISENSE: now also R29.2, V4.2; no longer RLOAD1.2
- net at U3.3 (~{CS}): now also U7.30 (D13)
- net at H3.3 (SDA): now also U7.22 (SDA); no longer U7.21 (SDA)
- net at H3.4 (SCL): now also U7.23 (SCL); no longer U7.22 (SCL)
- net at C8.1, M1.2 (+), U2.3 (VO): now also C19.1
- net at M1.3 (Tacho): now also U7.18 (D6)
- net at M1.4 (PWM): now also U7.17 (D8); no longer U7.16 (GND)
- net at H1.3 (SW): now also U7.26 (D9); no longer U7.25 (D9)
- net at H1.4 (DT): now also U7.25 (D7); no longer U7.24 (D7)
- net at H1.5 (CLK): now also U7.24 (D5); no longer U7.23 (D5)
- net at H2.5 (CLK): now also U7.27 (D10); no longer U7.26 (D10)
- net at H2.4 (DT): now also U7.28 (D11); no longer U7.27 (D11)
- net at H2.3 (SW): now also U7.29 (D12); no longer U7.28 (D12)
- net at U7.5 (A0): now also R27.1, TH1.2
- new net: R29.1, RLOAD1.2, V4.1
- new net: D1.2 (A), R28.2
Other:
- note added: "Heatsink Temp"
- note removed: "IN/~{OUT}"
- moved on the sheet: C11, C8, D11, M1, R22, R8, RLOAD1, U2

Commit message: WIP
Parts:
- removed C12: 100n, Capacitor_THT:C_Rect_L10.0mm_W2.5mm_P7.50mm_MKS4, symbol Device:C
- removed C6: 4700u, Capacitor_THT:CP_Radial_D18.0mm_P7.50mm, symbol Device:C_Polarized
- removed F1: 1A, Fuse:Fuseholder_Littelfuse_100_series_5x20mm, symbol Device:Fuse
- removed R13: 100, Resistor_THT:R_Axial_DIN0204_L3.6mm_D1.6mm_P7.62mm_Horizontal, symbol Device:R
- removed T1: 115V to 24V, symbol Device:Transformer_1P_1S
- added C6: 100n, Capacitor_THT:C_Rect_L10.0mm_W2.5mm_P7.50mm_MKS4, symbol Device:C
- C7: value 10p -> 100n; footprint (none) -> Capacitor_THT:C_Rect_L10.0mm_W2.5mm_P7.50mm_MKS4
Connections:
- net +28V: no longer U2.1 (VI), U4.1 (VI)
- net +36V: now also C6.1; no longer C5.1
- net GND: now also C7.2; no longer C4.2
- net +15V: now reaches C7.1
- net +15V: now also C4.2, C5.1, U2.1 (VI), U4.1 (VI), C6.2
Other:
- note removed: "1W"
- moved on the sheet: C4, C5, D4, D8

Commit message: WIP
Parts:
- added R13: 47k, symbol Device:R
- added RV7: 20k, symbol Device:R_Potentiometer
- Q2, Q5: footprint Package_TO_SOT_THT:TO-92_HandSolder -> Package_TO_SOT_THT:TO-92_Inline; symbol Simulation_SPICE:NPN -> Transistor_BJT:2N3904
- R26: value 47k -> 4.7k
- R3: value 10k -> 4.7k
- R7: value 3.9k -> 8.2k
- R9: value 22k -> 10k
Connections:
- net +28V: now also Q5.3 (C); no longer Q5.1 (C)
- net GND: now also C16.2, Q2.1 (E), R3.1, U5.2 (A); no longer C16.1, Q2.3 (E), U5.1 (K), U7.1 (RST)
- net ISENSE: now also RV7.2; no longer R3.1
- net VREF: now also C15.1, C16.1, R1.2, U5.1 (K), U6.8 (VDD/VREF)
- net at R26.2, SW1.1 (A), U1.12 (+): now also R13.1
- net at D11.1 (K): now also Q2.3 (C); no longer Q2.1 (C)
- net at M1.3 (Tacho): now also U7.20 (D0); no longer U7.18 (D6)
- net at R8.1: now also Q5.1 (E); no longer Q5.3 (E)
- new net: R13.2, RV7.1
Other:
- moved on the sheet: C11, C16, D1, D3, D9, H3, Q3, R11, R12, R15, R2, R26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

Commit message: WIP
Parts:
- removed C11: 100u, Capacitor_THT:CP_Radial_D8.0mm_P3.50mm, symbol Device:C_Polarized
- removed C18: 100n, Capacitor_THT:C_Rect_L10.0mm_W2.5mm_P7.50mm_MKS4, symbol Device:C
- removed D11: 1N4001, Diode_THT:D_DO-41_SOD81_P10.16mm_Horizontal, symbol Device:D
- removed D2: 1N4001, Diode_THT:D_DO-41_SOD81_P10.16mm_Horizontal, symbol Diode:1N4001
- removed D3: I_LIMIT_ON, Diode_THT:D_DO-35_SOD27_P5.08mm_Vertical_KathodeUp, symbol Device:LED
- removed D9: 1N4751ATR, Diode_THT:D_DO-41_SOD81_P10.16mm_Horizontal, symbol Device:D_Zener
- removed Q1: TIP121, Package_TO_SOT_THT:TO-220-3_Vertical, symbol Transistor_BJT:TIP121
- removed R11, R12, R9: 10k, Resistor_THT:R_Axial_DIN0204_L3.6mm_D1.6mm_P7.62mm_Horizontal, symbol Device:R
- removed R8: 1.5k, Resistor_THT:R_Axial_DIN0204_L3.6mm_D1.6mm_P7.62mm_Horizontal, symbol Device:R
- removed RLOAD1: 10k, symbol Device:R
- removed RV5: 20k, Potentiometer_THT:Potentiometer_Bourns_3339H_Vertical, symbol Device:R_Potentiometer
- removed RV7: 20k, symbol Device:R_Potentiometer
- removed unit 1 of U1
- removed V4: VSIN, symbol Simulation_SPICE:VSIN
- added C13: 1n, Capacitor_THT:C_Disc_D3.4mm_W2.1mm_P2.50mm, symbol Device:C
- added C17: 100n, Capacitor_THT:C_Disc_D3.4mm_W2.1mm_P2.50mm, symbol Device:C
- added D3: 1N4752A, Diode_THT:D_DO-41_SOD81_P5.08mm_Vertical_KathodeUp, symbol Diode:1N47xxA
- added D9: I_LIMIT_ON, Connector_PinHeader_2.54mm:PinHeader_1x02_P2.54mm_Vertical, symbol Device:LED
- added R21: 4.7k, Resistor_THT:R_Axial_DIN0204_L3.6mm_D1.6mm_P7.62mm_Horizontal, symbol Device:R
- added R25: 10k, Resistor_THT:R_Axial_DIN0204_L3.6mm_D1.6mm_P7.62mm_Horizontal, symbol Device:R
- added R26: 220, Resistor_THT:R_Axial_DIN0204_L3.6mm_D1.6mm_P7.62mm_Horizontal, symbol Device:R
- added R27: 0.05, Resistor_THT:R_Axial_DIN0207_L6.3mm_D2.5mm_P10.16mm_Horizontal, symbol Device:R
- added R30: 1k, Resistor_THT:R_Axial_DIN0204_L3.6mm_D1.6mm_P7.62mm_Horizontal, symbol Device:R
- added RV6: 10k, Potentiometer_THT:Potentiometer_Bourns_3339H_Vertical, symbol Device:R_Potentiometer
- added U8: INA225, Package_SO:VSSOP-8_3.0x3.0mm_P0.65mm, symbol Amplifier_Current:INA225
- C1: renamed from C6; footprint Capacitor_THT:C_Rect_L10.0mm_W2.5mm_P7.50mm_MKS4 -> Capacitor_THT:C_Disc_D3.4mm_W2.1mm_P2.50mm
- C11: renamed from C8; footprint Capacitor_THT:C_Rect_L10.0mm_W2.5mm_P7.50mm_MKS4 -> Capacitor_THT:C_Disc_D3.4mm_W2.1mm_P2.50mm
- C14: renamed from C2; value 10nf -> 1n; footprint Capacitor_THT:C_Rect_L10.0mm_W2.5mm_P7.50mm_MKS4 -> Capacitor_THT:C_Disc_D3.4mm_W2.1mm_P2.50mm
- C16: renamed from C14; footprint Capacitor_THT:C_Rect_L10.0mm_W2.5mm_P7.50mm_MKS4 -> Capacitor_THT:C_Disc_D3.4mm_W2.1mm_P2.50mm
- C2: renamed from C7; footprint Capacitor_THT:C_Rect_L10.0mm_W2.5mm_P7.50mm_MKS4 -> Capacitor_THT:C_Disc_D3.4mm_W2.1mm_P2.50mm
- C5: renamed from C9; footprint Capacitor_THT:C_Rect_L10.0mm_W2.5mm_P7.50mm_MKS4 -> Capacitor_THT:C_Disc_D3.4mm_W2.1mm_P2.50mm
- C6: renamed from C10; footprint Capacitor_THT:C_Rect_L10.0mm_W2.5mm_P7.50mm_MKS4 -> Capacitor_THT:C_Disc_D3.4mm_W2.1mm_P2.50mm
- C7: renamed from C3; footprint Capacitor_THT:C_Rect_L10.0mm_W2.5mm_P7.50mm_MKS4 -> Capacitor_THT:C_Disc_D3.4mm_W2.1mm_P2.50mm
- C9: renamed from C15; footprint Capacitor_THT:C_Rect_L10.0mm_W2.5mm_P7.50mm_MKS4 -> Capacitor_THT:C_Disc_D3.4mm_W2.1mm_P2.50mm
- R10: renamed from R15; value 10k -> 6.8k
- R13: value 47k -> 1.5k; footprint (none) -> Resistor_THT:R_Axial_DIN0204_L3.6mm_D1.6mm_P7.62mm_Horizontal
- R15: renamed from R26; value 4.7k -> 47k
- R22: renamed from R3; value 4.7k -> 8.2k
- R24: renamed from R10; value 10k -> 3k
- R29: value 10 -> 1k; footprint (none) -> Resistor_THT:R_Axial_DIN0204_L3.6mm_D1.6mm_P7.62mm_Horizontal; now in the parts list
- R6: value 0.5 -> 100; footprint Resistor_THT:R_Axial_Power_L20.0mm_W6.4mm_P25.40mm -> Resistor_THT:R_Axial_DIN0204_L3.6mm_D1.6mm_P7.62mm_Horizontal
- R9: renamed from R2; value 47k -> 10k
- RV5: renamed from RV3; value 22k -> 10k
- renumbered C16 to C10, C19 to C12, C17 to C15, C1 to C18, C4 to C3, C5 to C4, C13 to C8, D12 to D1, D5 to D10, D10 to D2, D1 to D4, D4 to D5, D8 to D7, D7 to D8, H3 to H1, H1 to H3, J2 to J1, J1 to J2, Q5 to Q1, R5 to R1, R23 to R11, R20 to R12, R24 to R14, R21 to R16, R25 to R18, R22 to R19, R14 to R2, R27 to R20, R4 to R23, R7 to R28, R16 to R3, R18 to R4, R19 to R5, R28 to R7, R1 to R8, RV6 to RV1, RV4 to RV2, RV1 to RV3, RV2 to RV4, U4 to U2, U5 to U3, U6 to U4, U2 to U5, U7 to U6, U3 to U7, V2 to V1, V1 to V2
Connections:
- net +28V: now also R6.2, D3.1 (K); no longer Q1.3 (C), Q3.3 (E), R7.1
- net +36V: now also R13.1, R6.1, R7.1, R27.1, U8.1 (IN+); no longer Q3.2 (C)
- net GND: now also C18.2, D10.2 (A), J1.1 (Pin_1), Q1.1 (E), R28.2, R29.2, C17.1, D3.2 (A), R26.2, R30.2, U8.2 (GND), U8.5 (GS0), U8.6 (GS1), U8.7 (REF); no longer Q2.1 (E), R6.2
- net ISENSE: now also R21.2, U8.4 (OUT); no longer C18.2, D10.2 (A), J1.1 (Pin_1), R28.2, R29.2, R6.1, U1.9 (-)
- net V+: now also Q3.3 (E)
- net at U1.8: now also R17.2, C13.2, R25.1
- net at R24.2: now also Q2.3 (C), Q3.1 (B)
- net at R15.2, SW1.1 (A), U1.12 (+): no longer R13.1
- net at R29.1: now also Q2.2 (B), R25.2
- net +12V: now reaches C11.1, C12.1, M1.2 (+), U5.3 (VO)
- net +12V: now also C17.2, U8.3 (V_{S})
- net at Q1.2 (B), R17.1: now also R30.1
- net at R13.2: now also D9.2 (A)
- net at R22.2, U1.13 (-): now also C14.2, RV6.2; no longer C14.1
- net at R24.1, U1.14: now also C14.1; no longer C14.2
- net at R10.1, R9.2: now also U1.9 (-), C13.1; no longer U1.10 (+)
- net at R23.1: now also RV6.1
- new net: Q3.2 (C), R27.2, U8.8 (IN-)
- new net: R21.1, U1.10 (+)
- new net: Q2.1 (E), R26.1
- new net: D9.1 (K), Q1.3 (C)
Other:
- note removed: "GAIN ADJ"
- note removed: "NOTE: This isn't the true output voltage, since it doesn't take the drop caused by the low side sense into account. But since we collect that drop for the current measurement, we can use it to recover the true output voltage in software."
- note removed: "PRE REGULATION"
- moved on the sheet: C14, C18, D10, J1, J2, R15, R22, R23, R28, U1C, U1E

Commit message: WIP
Parts:
- RV1, RV2, RV5, RV6: footprint Potentiometer_THT:Potentiometer_Bourns_3339H_Vertical -> Potentiometer_THT:TRIM_3362P-1-253LF
Connections:
- net at C13.2, R17.2, R25.1: now also U1.1; no longer U1.8
- net at C13.1, R10.1, R9.2: now also U1.2 (-); no longer U1.9 (-)
- net at R21.1: now also U1.3 (+); no longer U1.10 (+)
Changed lines of the file:
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@@
       (effects (font (size 1.27 1.27)) (justify right))
     )
-    (property "Footprint" "Potentiometer_THT:Potentiometer_Bourns_3339H_Vertical" (at 35.56 295.91 0)
+    (property "Footprint" "Potentiometer_THT:TRIM_3362P-1-253LF" (at 35.56 295.91 0)
       (effects (font (size 1.27 1.27)) hide)
     )
@@
       (effects (font (size 1.27 1.27)) (justify right))
     )
-    (property "Footprint" "Potentiometer_THT:Potentiometer_Bourns_3339H_Vertical" (at 94.615 134.62 0)
+    (property "Footprint" "Potentiometer_THT:TRIM_3362P-1-253LF" (at 94.615 134.62 0)
       (effects (font (size 1.27 1.27)) hide)
     )
@@
       (effects (font (size 1.27 1.27)))
     )
-    (property "Footprint" "Potentiometer_THT:Potentiometer_Bourns_3339H_Vertical" (at 17.78 255.27 0)
+    (property "Footprint" "Potentiometer_THT:TRIM_3362P-1-253LF" (at 17.78 255.27 0)
       (effects (font (size 1.27 1.27)) hide)
     )
@@
     )
   )
-  (symbol (lib_id "Amplifier_Operational:LM324") (at 151.765 91.44 0) (unit 3)
+  (symbol (lib_id "Amplifier_Operational:LM324") (at 151.765 91.44 0) (unit 1)
     (in_bom yes) (on_board yes) (dnp no)
     (property "Reference" "U1" (at 151.765 81.28 0)
@@
       (project "Lab Supply"
         (path "/f6cf3eae-48b8-48e0-9cfc-676f1a35373e"
-          (reference "U1") (unit 3)
+          (reference "U1") (unit 1)
         )
       )
@@
       (effects (font (size 1.27 1.27)))
     )
-    (property "Footprint" "Potentiometer_THT:Potentiometer_Bourns_3339H_Vertical" (at 189.865 129.54 0)
-      (effects (font (size 1.27 1.27)) hide)
-    )
+    (property "Footprint" "Potentiometer_THT:TRIM_3362P-1-253LF" (at 189.865 129.54 0)
+      (effects (font (size 1.27 1.27)) hide)
+    )

Commit message: WIP
Parts:
- added C19, C21: 100n, Capacitor_THT:C_Disc_D3.4mm_W2.1mm_P2.50mm, symbol Device:C
- added C20: 10u, Capacitor_THT:CP_Radial_D8.0mm_P3.50mm, symbol Device:C_Polarized
- added Q4: BD139, Package_TO_SOT_THT:TO-126-3_Vertical, symbol Transistor_BJT:BD139
- D1, D2: value 1N4001 -> SB140-E3/54
- U3: value LM4040DBZ-2.0 -> LM4040DBZ-4.1
Connections:
- net +12V: no longer C17.2, U8.3 (V_{S})
- net +28V: now also C20.1, C21.1, Q4.1 (E); no longer D3.1 (K), R6.2
- net +36V: now also Q3.2 (C), Q4.2 (C); no longer R27.1, U8.1 (IN+)
- net +5V: now also C17.2, U8.3 (V_{S})
- net GND: now also C19.2, C20.2, C21.2
- net V+: now also R27.2, U8.8 (IN-); no longer Q3.3 (E)
- net at R21.1, U1.3 (+): now also C19.1
- new net: Q3.3 (E), R27.1, U8.1 (IN+)
- new net: D3.1 (K), Q4.3 (B), R6.2
Other:
- moved on the sheet: Q3

Commit message: WIP
Parts:
- C10, C12, C15, C20, C8: footprint Capacitor_THT:CP_Radial_D8.0mm_P3.50mm -> Capacitor_THT:CP_Radial_D4.0mm_P1.50mm
Changed lines of the file:
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@@
       (effects (font (size 1.27 1.27)) (justify left))
     )
-    (property "Footprint" "Capacitor_THT:CP_Radial_D8.0mm_P3.50mm" (at 65.1002 121.92 0)
+    (property "Footprint" "Capacitor_THT:CP_Radial_D4.0mm_P1.50mm" (at 65.1002 121.92 0)
       (effects (font (size 1.27 1.27)) hide)
     )
@@
       (effects (font (size 1.27 1.27)) (justify left))
     )
-    (property "Footprint" "Capacitor_THT:CP_Radial_D8.0mm_P3.50mm" (at 113.9952 265.43 0)
+    (property "Footprint" "Capacitor_THT:CP_Radial_D4.0mm_P1.50mm" (at 113.9952 265.43 0)
       (effects (font (size 1.27 1.27)) hide)
     )
@@
       (effects (font (size 1.27 1.27)) (justify left))
     )
-    (property "Footprint" "Capacitor_THT:CP_Radial_D8.0mm_P3.50mm" (at 138.1252 353.06 0)
+    (property "Footprint" "Capacitor_THT:CP_Radial_D4.0mm_P1.50mm" (at 138.1252 353.06 0)
       (effects (font (size 1.27 1.27)) hide)
     )
@@
       (effects (font (size 1.27 1.27)))
     )
-    (property "Footprint" "Capacitor_THT:CP_Radial_D8.0mm_P3.50mm" (at 220.98 250.4948 0)
+    (property "Footprint" "Capacitor_THT:CP_Radial_D4.0mm_P1.50mm" (at 220.98 250.4948 0)
       (effects (font (size 1.27 1.27)) hide)
     )
@@
       (effects (font (size 1.27 1.27)) (justify left))
     )
-    (property "Footprint" "Capacitor_THT:CP_Radial_D8.0mm_P3.50mm" (at 80.9752 351.79 0)
-      (effects (font (size 1.27 1.27)) hide)
-    )
+    (property "Footprint" "Capacitor_THT:CP_Radial_D4.0mm_P1.50mm" (at 80.9752 351.79 0)
+      (effects (font (size 1.27 1.27)) hide)
+    )
